Commit message: results

File: my_bot/urdf/common_properties.xacro (robot description, xacro)
@@ -1,4 +1,4 @@
 <?xml version="1.0" ?>
-<robot name="xacro_properties" xmlns:xacro="http://www.ros.org/wiki/xacro">
+<robot name="xacro_properties" xmlns:xacro="http://ros.org/wiki/xacro">
   <!-- Init colour -->
   <material name="black">

File: my_bot/urdf/my_bot.xacro (robot description, xacro)
@@ -1,136 +1,121 @@
 <?xml version='1.0'?>
-<robot name="udacity_bot" xmlns:xacro="http://www.ros.org/wiki/xacro">
-  <xacro:include filename="$(find udacity_bot)/urdf/udacity_bot.gazebo"/>
+<robot name="my_bot" xmlns:xacro="http://www.ros.org/wiki/xacro">
+  <xacro:include filename="$(find my_bot)/urdf/my_bot.gazebo"/>
+  <xacro:include filename="$(find my_bot)/urdf/common_properties.xacro"/>
   <link name="robot_footprint"></link>
   <joint name="robot_footprint_joint" type="fixed">
-    <origin xyz="0 0 0" rpy="0 0 0" />
     <parent link="robot_footprint"/>
-    <child link="chassis" />
-  </joint>
-  <!-- Chassis Link -->
-  <link name='chassis'>
-    <pose>0 0 0.1 0 0 0</pose>
-    <inertial>
-      <mass value="15.0"/>
-      <origin xyz="0.0 0 0" rpy=" 0 0 0"/>
-      <inertia
-          ixx="0.1" ixy="0" ixz="0"
-          iyy="0.1" iyz="0"
-          izz="0.1"
-      />
-    </inertial>
-    <collision name='collision'>
-      <origin xyz="0 0 0" rpy=" 0 0 0"/>
-      <geometry>
-        <box size=".4 .4 .1"/>
-      </geometry>
-    </collision>
-    <visual name='chassis_visual'>
-      <origin xyz="0 0 0" rpy=" 0 0 0"/>
-      <geometry>
-        <box size=".4 .4 .1"/>
-      </geometry>
-      <material name="black">
-        <color rgba="0 0 0 1"/>
-      </material>
-    </visual>
-    <collision name='right_caster_collision'>
-      <origin xyz="0.15 -0.1 -0.05" rpy=" 0 0 0"/>
-      <geometry>
-        <sphere radius="0.0499"/>
-      </geometry>
-      <surface>
-        <friction>
-          <ode>
-            <mu>0</mu>
-            <mu2>0</mu2>
-            <slip1>1.0</slip1>
-            <slip2>1.0</slip2>
-          </ode>
-        </friction>
-      </surface>
-    </collision>
-    <visual name='right_caster_visual'>
-      <origin xyz="0.15 -0.1 -0.05" rpy=" 0 0 0"/>
-      <geometry>
-        <sphere radius="0.0499"/>
-      </geometry>
-    </visual>
-    <collision name='left_caster_collision'>
-      <origin xyz="0.15 0.1 -0.05" rpy=" 0 0 0"/>
-      <geometry>
-        <sphere radius="0.0499"/>
-      </geometry>
-      <surface>
-        <friction>
-          <ode>
-            <mu>0</mu>
-            <mu2>0</mu2>
-            <slip1>1.0</slip1>
-            <slip2>1.0</slip2>
-          </ode>
-        </friction>
-      </surface>
-    </collision>
-    <visual name='left_caster_visual'>
-      <origin xyz="0.15 0.1 -0.05" rpy=" 0 0 0"/>
-      <geometry>
-        <sphere radius="0.0499"/>
-      </geometry>
-    </visual>
-  </link>
-  <!-- Left Wheel Link -->
-  <link name="left_wheel">
-    <inertial>
-      <mass value="5.0"/>
-      <origin xyz="0 0 0" rpy="0 1.5707 1.5707"/>
-      <inertia
-          ixx="0.1" ixy="0" ixz="0"
-          iyy="0.1" iyz="0"
-          izz="0.1"
-      />
-    </inertial>
-    <visual>
-      <geometry>
-        <cylinder length="0.05" radius="0.1"/>
-      </geometry>
-      <origin xyz="0 0 0" rpy="0 1.5707 1.5707"/>
-      <material name="white">
-        <color rgba="1 1 1 1"/>
-      </material>
-    </visual>
-    <collision>
-      <geometry>
-        <cylinder length="0.05" radius="0.1"/>
-      </geometry>
-      <origin xyz="0 0 0" rpy="0 1.5707 1.5707"/>
-    </collision>
-  </link>
-  <!-- Right Wheel Link -->
-  <link name="right_wheel">
-    <inertial>
-      <mass value="5.0"/>
-      <origin xyz="0 0 0" rpy="0 1.5707 1.5707"/>
-      <inertia
-          ixx="0.1" ixy="0" ixz="0"
-          iyy="0.1" iyz="0"
-          izz="0.1"
-      />
-    </inertial>
-    <visual>
-      <geometry>
-        <cylinder length="0.05" radius="0.1"/>
-      </geometry>
-      <origin xyz="0 0 0" rpy="0 1.5707 1.5707"/>
-      <material name="white">
-        <color rgba="1 1 1 1"/>
-      </material>
-    </visual>
-    <collision>
-      <geometry>
-        <cylinder length="0.05" radius="0.1"/>
-      </geometry>
-      <origin xyz="0 0 0" rpy="0 1.5707 1.5707"/>
-    </collision>
+    <child link="chasis" />
+    <origin xyz="0 0 0.0122" rpy="0 0 0"/>
+  </joint>
+  <link name="chasis">
+    <visual>
+      <origin xyz="-0.035 0 0.0" rpy="0 0 0"/>
+      <geometry>
+        <mesh filename="package://my_bot/meshes/platform_mesh.stl" scale="0.001 0.001 0.001"/>
+      </geometry>
+      <material name="light_black"/>
+    </visual>
+    <collision>
+      <origin xyz="-0.035 0 0.02901" rpy="0 0 0"/>
+      <geometry>
+        <box size="0.220 0.220 0.05802"/>
+      </geometry>
+    </collision>
+    <inertial>
+      <origin xyz="0 0 0" rpy="0 0 0"/>
+    <mass value="0.881e+00"/>
+    <inertia ixx="3.0e-03" ixy="0" ixz="0"
+         iyy="3.0e-03" iyz="0"
+         izz="6.0e-03" />
+    </inertial>
+  </link>
+  <link name="wheel_left_link">
+    <visual>
+      <origin xyz="0 0 -0.0085" rpy="0 1.57 0"/>
+      <geometry>
+        <mesh filename="package://my_bot/meshes/wheel_mesh.stl" scale="0.001 0.001 0.001"/>
+      </geometry>
+      <material name="dark"/>
+    </visual>
+    <collision>
+      <origin xyz="0 0 0.0045" rpy="0 0 0"/>
+      <geometry>
+        <cylinder length="0.026" radius="0.0325"/>
+      </geometry>
+    </collision>
+    <inertial>
+      <origin xyz="0 0 0" />
+    <mass value="3.3e-02" />
+      <inertia ixx="1e-05" ixy="0.0" ixz="0.0"
+               iyy="1e-05" iyz="0.0"
+               izz="1e-05" />
+    </inertial>
+  </link>
+  <link name="wheel_right_link">
+  <visual>
+    <origin xyz="0 0 0.0085" rpy="0 -1.57 0"/>
+    <geometry>
+    <mesh filename="package://my_bot/meshes/wheel_mesh.stl" scale="0.001 0.001 0.001"/>
+    </geometry>
+    <material name="dark"/>
+  </visual>
+  <collision>
+    <origin xyz="0 0 -0.0045" rpy="0 0 0"/>
+    <geometry>
+    <cylinder length="0.026" radius="0.0325"/>
+    </geometry>
+  </collision>
+  <inertial>
+    <origin xyz="0 0 0" />
+    <mass value="3.3e-02" />
+      <inertia ixx="1e-05" ixy="0.0" ixz="0.0"
+               iyy="1e-05" iyz="0.0"
+               izz="1e-05" />
+    </inertial>
+  </link>
+  <link name="caster_back_right_link">
+  <visual>
+    <origin xyz="0 0 0" rpy="0 0 0"/>
+    <geometry>
+    <mesh filename="package://my_bot/meshes/caster_ball_mesh.stl" scale="0.001 0.001 0.001"/>
+    </geometry>
+    <material name="white"/>
+  </visual>
+  <collision>
+    <origin xyz="0.000575 0 0" rpy="0 0 0"/>
+    <geometry>
+    <box size="0.01385 0.013 0.013"/>
+    </geometry>
+  </collision>
+  <inertial>
+    <origin xyz="0 0 0" />
+    <mass value="8.37e-03" />
+      <inertia ixx="1e-03" ixy="0.0" ixz="0.0"
+               iyy="1e-03" iyz="0.0"
+               izz="1e-03" />
+    </inertial>
+  </link>
+  <link name="caster_back_left_link">
+  <visual>
+    <origin xyz="0 0 0" rpy="0 0 0"/>
+    <geometry>
+    <mesh filename="package://my_bot/meshes/caster_ball_mesh.stl" scale="0.001 0.001 0.001"/>
+    </geometry>
+    <material name="white"/>
+  </visual>
+  <collision>
+    <origin xyz="0.000575 0 0" rpy="0 0 0"/>
+    <geometry>
+    <box size="0.01385 0.013 0.013"/>
+    </geometry>
+  </collision>
+  <inertial>
+    <origin xyz="0 0 0" />
+    <mass value="8.37e-03" />
+      <inertia ixx="1e-03" ixy="0.0" ixz="0.0"
+               iyy="1e-03" iyz="0.0"
+               izz="1e-03" />
+    </inertial>
   </link>
   <!-- Camera Link -->
@@ -147,5 +132,5 @@
     <visual>
       <geometry>
-        <box size="0.05 0.05 0.05"/>
+        <box size="0.025 0.025 0.025"/>
       </geometry>
       <origin xyz="0 0 0" rpy="0 0 0"/>
@@ -156,5 +141,5 @@
     <collision>
       <geometry>
-        <box size="0.05 0.05 0.05"/>
+        <box size="0.025 0.025 0.025"/>
       </geometry>
       <origin xyz="0 0 0" rpy="0 0 0"/>
@@ -174,11 +159,11 @@
     <visual>
       <geometry>
-        <mesh filename="package://udacity_bot/meshes/hokuyo.dae"/>
-      </geometry>
-      <origin xyz="0 0 0" rpy="0 0 0"/>
-    </visual>
-    <collision>
-      <geometry>
-        <box size="0.1 0.1 0.1"/>
+        <mesh filename="package://my_bot/meshes/hokuyo.dae"/>
+      </geometry>
+      <origin xyz="0 0 0" rpy="0 0 0"/>
+    </visual>
+    <collision>
+      <geometry>
+        <box size="0.05 0.05 0.05"/>
       </geometry>
       <origin xyz="0 0 0" rpy="0 0 0"/>
@@ -186,29 +171,35 @@
   </link>
   <!-- Joints -->
-  <joint type="continuous" name="left_wheel_hinge">
-    <origin xyz="-0.15 0.25 0" rpy="0 0 0"/>
-    <child link="left_wheel"/>
-    <parent link="chassis"/>
-    <axis xyz="0 1 0" rpy="0 0 0"/>
-    <limit effort="10000" velocity="1000"/>
-    <joint_properties damping="1.0" friction="1.0"/>
-  </joint>
-  <joint type="continuous" name="right_wheel_hinge">
-    <origin xyz="-0.15 -0.25 0" rpy="0 0 0"/>
-    <child link="right_wheel"/>
-    <parent link="chassis"/>
-    <axis xyz="0 1 0" rpy="0 0 0"/>
-    <limit effort="10000" velocity="1000"/>
-    <joint_properties damping="1.0" friction="1.0"/>
+  <joint name="wheel_right_joint" type="continuous">
+    <parent link="chasis"/>
+    <child link="wheel_right_link"/>
+    <origin xyz="0.015 0.09975 0.0188" rpy="-1.57 0 0"/>
+    <axis xyz="0 0 1"/>
+  </joint>
+  <joint name="wheel_left_joint" type="continuous">
+    <parent link="chasis"/>
+    <child link="wheel_left_link"/>
+    <origin xyz="0.015 -0.09975 0.0188" rpy="-1.57 0 0"/>
+    <axis xyz="0 0 1"/>
+  </joint>
+  <joint name="caster_back_right_joint" type="fixed">
+  <parent link="chasis"/>
+  <child link="caster_back_right_link"/>
+  <origin xyz="-0.133 0.053 -0.0075" rpy="-1.57 0 0"/>
+  </joint>
+  <joint name="caster_back_left_joint" type="fixed">
+  <parent link="chasis"/>
+  <child link="caster_back_left_link"/>
+  <origin xyz="-0.133 -0.053 -0.0075" rpy="-1.57 0 0"/>
   </joint>
   <joint type="fixed" name="camera_joint">
-    <origin xyz="0.2 0 0" rpy="0 0 0"/>
+    <origin xyz="-0.12 0 0.075" rpy="0 0 3.14"/>
     <child link="camera"/>
-    <parent link="chassis"/>
+    <parent link="chasis"/>
   </joint>
   <joint type="fixed" name="hokuyo_joint">
-    <origin xyz="0.15 0 0.1" rpy="0 0 0"/>
+    <origin xyz="0.02 0 0.1" rpy="0 0 3.14"/>
     <child link="hokuyo"/>
-    <parent link="chassis"/>
+    <parent link="chasis"/>
   </joint>
 </robot>
